File: pcb/lavender58.kicad_sch (KiCad schematic)
At the start: 124 parts, among them U1 xiao-ble, U2 xiao-ble

Commit message: finished lavender58 board
Parts:
- removed DL1, DL10, DL11, DL12, DL13, DL14, DL15, DL16, DL17, DL18, DL19, DL2, DL20, DL21, DL22, DL23, DL24, DL25, DL26, DL27, DL28, DL29, DL3, DL4, DL5, DL6, DL7, DL8, DL9, DR1, DR10, DR11, DR12, DR13, DR14, DR15, DR16, DR17, DR18, DR19, DR2, DR20, DR21, DR22, DR23, DR24, DR25, DR26, DR27, DR28, DR29, DR3, DR4, DR5, DR6, DR7, DR8, DR9: D_Small, Diode_SMD:D_SOD-123, symbol Device:D_Small
- removed SWL1, SWL10, SWL11, SWL12, SWL13, SWL14, SWL15, SWL16, SWL17, SWL18, SWL19, SWL2, SWL20, SWL21, SWL22, SWL23, SWL24, SWL25, SWL26, SWL27, SWL28, SWL29, SWL3, SWL4, SWL5, SWL6, SWL7, SWL8, SWL9, SWR1, SWR10, SWR11, SWR12, SWR13, SWR14, SWR15, SWR16, SWR17, SWR18, SWR19, SWR2, SWR20, SWR21, SWR22, SWR23, SWR24, SWR25, SWR26, SWR27, SWR28, SWR29, SWR3, SWR4, SWR5, SWR6, SWR7, SWR8, SWR9: SW_Push_45deg, PCM_marbastlib-choc:SW_choc_v1_1u, symbol Switch:SW_Push_45deg
- added KL1, KL10, KL11, KL12, KL13, KL14, KL15, KL16, KL17, KL18, KL19, KL2, KL20, KL21, KL22, KL23, KL24, KL25, KL26, KL27, KL28, KL29, KL3, KL4, KL5, KL6, KL7, KL8, KL9, KR1, KR10, KR11, KR12, KR13, KR14, KR15, KR16, KR17, KR18, KR19, KR2, KR20, KR21, KR22, KR23, KR24, KR25, KR26, KR27, KR28, KR29, KR3, KR4, KR5, KR6, KR7, KR8, KR9: diode-choc, lavender58lib:pg1350-D, symbol lavender58:diode-choc
- BAT+1, BAT+2, BATGND1, BATGND2: footprint Connector_Wire:SolderWirePad_1x01_SMD_2x4mm -> Connector_Wire:SolderWirePad_1x01_SMD_1.5x3mm
- PSW1, PSW2: footprint TOTEMlib:MSK12C02 -> lavender58lib:CUS-12TB_NDC
- U1, U2: footprint TOTEMlib:xiao-ble-smd-cutout -> lavender58lib:xiao-ble-smd-cutout
Connections:
- net COL0_L: now also KL1.2, KL13.2, KL19.2, KL7.2
- net COL0_R: now also KR1.2, KR13.2, KR19.2, KR7.2
- net COL1_L: now also KL14.2, KL2.2, KL20.2, KL25.2, KL8.2
- net COL1_R: now also KR14.2, KR2.2, KR20.2, KR25.2, KR8.2
- net COL2_L: now also KL15.2, KL21.2, KL26.2, KL3.2, KL9.2
- net COL2_R: now also KR15.2, KR21.2, KR26.2, KR3.2, KR9.2
- net COL3_L: now also KL10.2, KL16.2, KL22.2, KL27.2, KL4.2
- net COL3_R: now also KR10.2, KR16.2, KR22.2, KR27.2, KR4.2
- net COL4_L: now also KL11.2, KL17.2, KL23.2, KL28.2, KL5.2
- net COL4_R: now also KR11.2, KR17.2, KR23.2, KR28.2, KR5.2
- net COL5_L: now also KL12.2, KL18.2, KL24.2, KL29.2, KL6.2
- net COL5_R: now also KR12.2, KR18.2, KR24.2, KR29.2, KR6.2
- net ROW0_L: now also KL1.1, KL2.1, KL3.1, KL4.1, KL5.1, KL6.1
- net ROW0_R: now also KR1.1, KR2.1, KR3.1, KR4.1, KR5.1, KR6.1
- net ROW1_L: now also KL10.1, KL11.1, KL12.1, KL7.1, KL8.1, KL9.1
- net ROW1_R: now also KR10.1, KR11.1, KR12.1, KR7.1, KR8.1, KR9.1
- net ROW2_L: now also KL13.1, KL14.1, KL15.1, KL16.1, KL17.1, KL18.1
- net ROW2_R: now also KR13.1, KR14.1, KR15.1, KR16.1, KR17.1, KR18.1
- net ROW3_L: now also KL19.1, KL20.1, KL21.1, KL22.1, KL23.1, KL24.1
- net ROW3_R: now also KR19.1, KR20.1, KR21.1, KR22.1, KR23.1, KR24.1
- net ROW4_L: now also KL25.1, KL26.1, KL27.1, KL28.1, KL29.1
- net ROW4_R: now also KR25.1, KR26.1, KR27.1, KR28.1, KR29.1
